File: DRXDaughterboard.kicad_sch (KiCad schematic)
At the start: 11 parts, among them J1 Samtec_ASP-134488-01, J2 Samtec_ASP-134488-01, J3 Conn_02x12_Odd_Even, J4 Samtec_ASP-134488-01, J5 Samtec_ASP-134488-01, J6 Conn_02x06_Odd_Even, J7 Samtec_ASP-134486-01, J8 Samtec_ASP-134486-01, U1 SN74LVC2T45DCUR

Commit message: Work on swapping fclk and lclk pins on J1/J4.  Add a power LED running powered by the +3.3V.  Rename.
Parts:
- added D1: LED, LED_SMD:LED_1206_3216Metric_Pad1.42x1.75mm_HandSolder, symbol Device:LED
- added R1: 324, Resistor_SMD:R_0805_2012Metric_Pad1.20x1.40mm_HandSolder, symbol Device:R_US
- J6: now not fitted
Connections:
- net +3.3VP: now also R1.1
- net FMC0_FCLKA_N: now also J1.H5 (Pin_5); no longer J1.D5 (Pin_5)
- net FMC0_FCLKA_P: now also J1.H4 (Pin_4); no longer J1.D4 (Pin_4)
- net FMC0_LCLKA_N: now also J1.D5 (Pin_5); no longer J1.H5 (Pin_5)
- net FMC0_LCLKA_P: now also J1.D4 (Pin_4); no longer J1.H4 (Pin_4)
- net FMC1_FCLKA_N: now also J1.G3 (Pin_3); no longer J4.D5 (Pin_5)
- net FMC1_FCLKA_P: now also J1.G2 (Pin_2); no longer J4.D4 (Pin_4)
- net FMC1_LCLKA_N: now also J4.D5 (Pin_5); no longer J1.G3 (Pin_3)
- net FMC1_LCLKA_P: now also J4.D4 (Pin_4); no longer J1.G2 (Pin_2)
- net GND: now also D1.1 (K)
- new net: D1.2 (A), R1.2

Commit message: Version update.  Add datasheets.  DNP on J7/J8.
Parts:
- J7, J8: now not fitted
Other:
- company: (none) -> University of New Mexico
- title: (none) -> ZCU102 Daughter Board
Changed lines of the file:
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@@
 	(generator_version "8.0")
 	(paper "A1")
+	(title_block
+		(title "ZCU102 Daughter Board")
+		(date "2026-07-07")
+		(rev "2.0")
+		(company "University of New Mexico")
+		(comment 1 "Long Wavelength Array")
+	)
 	(junction
 		(at 273.05 116.84)
@@
 		(in_bom yes)
 		(on_board yes)
-		(dnp no)
+		(dnp yes)
 		(fields_autoplaced yes)
 		(property "Reference" "J8"
@@
 		(in_bom yes)
 		(on_board yes)
-		(dnp no)
+		(dnp yes)
 		(fields_autoplaced yes)
 		(property "Reference" "J7"
@@
 		(in_bom yes)
 		(on_board yes)
-		(dnp no)
+		(dnp yes)
 		(fields_autoplaced yes)
 		(property "Reference" "J8"
@@
 		(in_bom yes)
 		(on_board yes)
-		(dnp no)
+		(dnp yes)
 		(fields_autoplaced yes)
 		(property "Reference" "J7"
@@
 		(in_bom yes)
 		(on_board yes)
-		(dnp no)
+		(dnp yes)
 		(fields_autoplaced yes)
 		(property "Reference" "J7"
@@
 			)
 		)
-		(property "Datasheet" "~"
+		(property "Datasheet" "https://www.kingbrightusa.com/images/catalog/SPEC/APT3216LVBC-D.pdf"
 			(at 375.92 120.65 0)
 			(effects
@@
 			)
 		)
-		(property "Description" "Kingbrite APTD3216LCGCK"
+		(property "Description" "Kingbright APT3216LVBC/D (LED BLUE CLEAR 2SMD)"
 			(at 375.92 120.65 0)
 			(effects
@@
 		(in_bom yes)
 		(on_board yes)
-		(dnp no)
+		(dnp yes)
 		(fields_autoplaced yes)
 		(property "Reference" "J8"
@@
 		(in_bom yes)
 		(on_board yes)
-		(dnp no)
+		(dnp yes)
 		(fields_autoplaced yes)
 		(property "Reference" "J7"
@@
 			)
 		)
-		(property "Description" ""
+		(property "Description" "TI SN74LVC2T45DCUR"
 			(at 408.94 45.72 0)
 			(effects
@@
 		(in_bom yes)
 		(on_board yes)
-		(dnp no)
+		(dnp yes)
 		(fields_autoplaced yes)
 		(property "Reference" "J7"
@@
 		(in_bom yes)
 		(on_board yes)
-		(dnp no)
+		(dnp yes)
 		(fields_autoplaced yes)
 		(property "Reference" "J7"
@@
 		(in_bom yes)
 		(on_board yes)
-		(dnp no)
+		(dnp yes)
 		(fields_autoplaced yes)
 		(property "Reference" "J7"
@@
 		(in_bom yes)
 		(on_board yes)
-		(dnp no)
+		(dnp yes)
 		(fields_autoplaced yes)
 		(property "Reference" "J8"
@@
 		(in_bom yes)
 		(on_board yes)
-		(dnp no)
+		(dnp yes)
 		(fields_autoplaced yes)
 		(property "Reference" "J8"
@@
 		(in_bom yes)
 		(on_board yes)
-		(dnp no)
+		(dnp yes)
 		(fields_autoplaced yes)
 		(property "Reference" "J8"
@@
 		(in_bom yes)
 		(on_board yes)
-		(dnp no)
+		(dnp yes)
 		(fields_autoplaced yes)
 		(property "Reference" "J7"
@@
 		(in_bom yes)
 		(on_board yes)
-		(dnp no)
+		(dnp yes)
 		(fields_autoplaced yes)
 		(property "Reference" "J8"
@@
 		(in_bom yes)
 		(on_board yes)
-		(dnp no)
+		(dnp yes)
 		(fields_autoplaced yes)
 		(property "Reference" "J8"
@@
 			)
 		)
-		(property "Datasheet" "~"
+		(property "Datasheet" "https://www.yageo.com/upload/media/product/products/datasheet/rchip/PYu-RC_Group_51_RoHS_L_12.pdf"
 			(at 368.3 120.65 0)
 			(effects
@@
 			)
 		)
-		(property "Description" "Yaego RC0805FR-07324RL"
+		(property "Description" "Yageo RC0805FR-07324RL (RES 324 OHM 1% 1/8W 0805)"
 			(at 368.3 120.65 0)
 			(effects
@@
 		(in_bom yes)
 		(on_board yes)
-		(dnp no)
+		(dnp yes)
 		(fields_autoplaced yes)
 		(property "Reference" "J8"
@@
 		(in_bom yes)
 		(on_board yes)
-		(dnp no)
+		(dnp yes)
 		(fields_autoplaced yes)
 		(property "Reference" "J7"
@@
 		(in_bom yes)
 		(on_board yes)
-		(dnp no)
+		(dnp yes)
 		(fields_autoplaced yes)
 		(property "Reference" "J7"
@@
 		(in_bom yes)
 		(on_board yes)
-		(dnp no)
+		(dnp yes)
 		(fields_autoplaced yes)
 		(property "Reference" "J8"
@@
 			)
 		)
-		(property "Datasheet" "~"
+		(property "Datasheet" "https://www.samsungsem.com/resources/file/global/support/product_catalog/MLCC_2512.pdf"
 			(at 416.56 31.75 0)
 			(effects
@@
 			)
 		)
-		(property "Description" ""
+		(property "Description" "Samsung CL31B104KBCNFNC (CAP 100nF 1206)"
 			(at 416.56 31.75 0)
 			(effects
@@
 			)
 		)
-		(property "Datasheet" "~"
+		(property "Datasheet" "https://www.samsungsem.com/resources/file/global/support/product_catalog/MLCC_2512.pdf"
 			(at 401.32 31.75 0)
 			(effects
@@
 			)
 		)
-		(property "Description" ""
+		(property "Description" "Samsaung CL31B104KBCNFNC (CAP 100nF 1206)"
 			(at 401.32 31.75 0)
 			(effects
